Commit message: chore: inertia and mass updated

File: waver_description/urdf/lidar.xacro (robot description, xacro)
@@ -7,6 +7,5 @@
             <mass value="${mass_lidar}" />
             <origin xyz="0 0 0" rpy="0 0 0" />
-            <inertia ixx="1.3010226e-05" iyy="1.6209553e-05" izz="2.1055697e-05" ixy="0.0" iyz="0.0"
-                ixz="0.0" />
+            <inertia ixx="1.1969407982864896e-05" iyy="1.4912788506851203e-05" izz="1.9371239273809308e-05" ixy="0.0" iyz="0.0" ixz="0.0" />
         </inertial>
         <visual>

Commit message: feat(waver_description): urdf rasp pi camera module added

File: waver_description/urdf/lidar.xacro (robot description, xacro)
@@ -3,5 +3,5 @@
     <xacro:include filename="$(find waver_description)/urdf/materials.xacro" />
     <xacro:include filename="$(find waver_description)/urdf/util.xacro" />
-    <link name="${lidar_link}">
+    <link name="lidar_link">
         <inertial>
             <mass value="${mass_lidar}" />
@@ -26,7 +26,7 @@
         <origin xyz="0.04 0 ${base_to_top + 0.025}" rpy="0 0 0" />
         <parent link="top_shell_link" />
-        <child link="${lidar_link}" />
+        <child link="lidar_link" />
     </joint>
-    <gazebo reference="${lidar_link}">
+    <gazebo reference="lidar_link">
         <material>Gazebo/Black</material>
         <sensor name="${lidar_model}" type="ray">

File: waver_description/urdf/util.xacro (robot description, xacro)
@@ -92,5 +92,4 @@
     <xacro:property name="mass_lidar" value="0.046" />
     <xacro:property name="lidar_model" value="HLS-LFCD-LDS" />
-    <xacro:property name="lidar_link" value="lidar_link" />
     <xacro:property name="lidar_samples" value="720" />
     <xacro:property name="lidar_max_range" value="12.0" />
@@ -100,3 +99,6 @@
     <xacro:property name="lidar_frequency" value="10" />
     <xacro:property name="lidar_transform" value="0 0 0 0 0 0" />
+    <!-- Rasp Pi Camera specifications -->
+    <xacro:property name="rasp_pi_camera_mass" value="0.0035" />
+    <xacro:property name="camera_scale" value="0.0005 0.0005 0.0005" />
 </robot>

File: waver_description/urdf/waver.xacro (robot description, xacro)
@@ -7,4 +7,5 @@
   <xacro:include filename="$(find waver_description)/urdf/lidar.xacro" />
   <xacro:include filename="$(find waver_description)/urdf/imu.xacro" />
+  <xacro:include filename="$(find waver_description)/urdf/rasp_pi_camera.xacro" />
   <!-- ******************************* Links ******************************* -->
   <link name="base_footprint"></link>
