Commit message: feat(description | rviz): urdf and gazebo plugin depth camera (zed x mini) added

File: waver_description/urdf/util.xacro (robot description, xacro)
@@ -102,3 +102,6 @@
     <xacro:property name="rasp_pi_camera_mass" value="0.0035" />
     <xacro:property name="camera_scale" value="0.0005 0.0005 0.0005" />
+    <!-- ZED X Mini Stereo Camera specifications -->
+    <xacro:property name="zed_x_mini_mass" value="0.015" />
+    <xacro:property name="zed_x_mini_scale" value="1 1 1" />
 </robot>

File: waver_description/urdf/waver.xacro (robot description, xacro)
@@ -1,4 +1,5 @@
 <?xml version="1.0"?>
 <robot name="waver" xmlns:xacro="http://www.ros.org/wiki/xacro">
+  <xacro:arg name="camera_type" default="raspi" />
   <xacro:include filename="$(find waver_description)/urdf/materials.xacro" />
   <xacro:include filename="$(find waver_description)/urdf/util.xacro" />
@@ -7,5 +8,10 @@
   <xacro:include filename="$(find waver_description)/urdf/lidar.xacro" />
   <xacro:include filename="$(find waver_description)/urdf/imu.xacro" />
-  <xacro:include filename="$(find waver_description)/urdf/rasp_pi_camera.xacro" />
+  <xacro:if value="${'$(arg camera_type)' == 'raspi'}">
+    <xacro:include filename="$(find waver_description)/urdf/rasp_pi_camera.xacro" />
+  </xacro:if>
+  <xacro:if value="${'$(arg camera_type)' == 'depth'}">
+    <xacro:include filename="$(find waver_description)/urdf/depth_camera_zedxm.xacro" />
+  </xacro:if>
   <!-- ******************************* Links ******************************* -->
   <link name="base_footprint"></link>
