Commit message: chore(desc): inertial and collisions updated for some links

File: waver_description/urdf/depth_camera_zedxm.xacro (robot description, xacro)
@@ -17,7 +17,7 @@
         </visual>
         <collision>
-            <origin xyz="0 0 0" rpy="0 0 0" />
+            <origin xyz="0 0 ${base_to_top - 0.039}" rpy="0 0 0" />
             <geometry>
-                <mesh filename="package://waver_description/meshes/zedxm.stl" scale="${zed_x_mini_scale}" />
+                <box size="${zed_x_mini_dimensions}" />
             </geometry>
         </collision>

File: waver_description/urdf/imu.xacro (robot description, xacro)
@@ -4,9 +4,4 @@
     <xacro:include filename="$(find waver_description)/urdf/util.xacro" />
     <link name="imu_link">
-        <inertial>
-            <mass value="${mass_imu}" />
-            <origin xyz="${mass_center_imu}" rpy="0 0 ${pi/2}" />
-            <inertia ixx="4.297064285474092e-13" iyy="4.199442581059605e-13" izz="7.142756866533696e-13" ixy="0.0" iyz="0.0" ixz="0.0" />
-        </inertial>
         <visual>
             <origin xyz="${position_imu}" rpy="0 0 ${pi/2}" />
@@ -16,10 +11,4 @@
             <xacro:dark_green_material />
         </visual>
-        <collision>
-            <origin xyz="${position_imu}" rpy="0 0 ${pi/2}" />
-            <geometry>
-                <mesh filename="package://waver_description/meshes/board_link.stl" scale="${scale}" />
-            </geometry>
-        </collision>
     </link>
     <joint name="top_imu_joint" type="fixed">

File: waver_description/urdf/lidar.xacro (robot description, xacro)
@@ -17,7 +17,7 @@
         </visual>
         <collision>
-            <origin xyz="0 0 -0.027" rpy="0 0 ${pi/2}" />
+            <origin xyz="0 0 -0.0107" rpy="0 0 0" />
             <geometry>
-                <mesh filename="package://waver_description/meshes/LD19.stl" scale="${scale}" />
+                <box size="0.0383 0.0383 0.030" />
             </geometry>
         </collision>

File: waver_description/urdf/rasp_pi_camera.xacro (robot description, xacro)
@@ -4,10 +4,4 @@
     <xacro:include filename="$(find waver_description)/urdf/util.xacro" />
     <link name="rasp_pi_camera_link">
-        <inertial>
-            <mass value="${rasp_pi_camera_mass}" />
-            <origin xyz="0 0 0" rpy="0 0 0" />
-            <inertia ixx="8.188544198245058e-07" iyy="1.3934609636775025e-06"
-                izz="8.837267894803364e-07" ixy="0" iyz="0" ixz="0" />
-        </inertial>
         <visual>
             <origin xyz="0 0.0125 0" rpy="0 0 ${-pi/2}" />
@@ -19,8 +13,7 @@
         </visual>
         <collision>
-            <origin xyz="0 0.0125 0" rpy="0 0 ${-pi/2}" />
+            <origin xyz="0.005 0 -0.012" rpy="0 0 0" />
             <geometry>
-                <mesh filename="package://waver_description/meshes/rasp_pi_camera.stl"
-                    scale="${camera_scale}" />
+                <box size="0.01 0.025 0.023" />
             </geometry>
         </collision>

File: waver_description/urdf/util.xacro (robot description, xacro)
@@ -105,3 +105,4 @@
     <xacro:property name="zed_x_mini_mass" value="0.015" />
     <xacro:property name="zed_x_mini_scale" value="1 1 1" />
+    <xacro:property name="zed_x_mini_dimensions" value="0.030 0.093 0.0315" />
 </robot>

File: waver_description/urdf/waver.xacro (robot description, xacro)
@@ -66,10 +66,4 @@
   </link>
   <link name="accessories_link">
-    <inertial>
-      <mass value="${mass_acces}" />
-      <origin xyz="${mass_center_acces}" rpy="0 0 ${pi/2}" />
-      <inertia ixx="1.284177729497181e-13" iyy="4.1792730400878273e-13" izz="4.1792732165684473e-13"
-        ixy="0.0" iyz="0.0" ixz="0.0" />
-    </inertial>
     <visual>
       <origin xyz="${position_acces}" rpy="0 0 ${pi/2}" />
@@ -87,10 +81,4 @@
   </link>
   <link name="accessories1_link">
-    <inertial>
-      <mass value="${mass_acces1}" />
-      <origin xyz="${mass_center_acces1}" rpy="0 0 ${pi/2}" />
-      <inertia ixx="8.4505377139432e-14" iyy="3.769648155305237e-13" izz="3.769601126710828e-13"
-        ixy="0.0" iyz="0.0" ixz="0.0" />
-    </inertial>
     <visual>
       <origin xyz="${position_acces1}" rpy="0 0 ${pi/2}" />
@@ -100,18 +88,6 @@
       <xacro:black_material />
     </visual>
-    <collision>
-      <origin xyz="${position_acces1}" rpy="0 0 ${pi/2}" />
-      <geometry>
-        <mesh filename="package://waver_description/meshes/accessories1_link.stl" scale="${scale}" />
-      </geometry>
-    </collision>
   </link>
   <link name="oled_screen_link">
-    <inertial>
-      <mass value="${mass_screen}" />
-      <origin xyz="${mass_center_screen}" rpy="0 0 ${pi/2}" />
-      <inertia ixx="2.2613546657562738e-14" iyy="1.821435448519393e-13" izz="1.9313666847229008e-13"
-        ixy="0.0" iyz="0.0" ixz="0.0" />
-    </inertial>
     <visual>
       <origin xyz="${position_screen}" rpy="0 0 ${pi/2}" />
@@ -121,10 +97,4 @@
       <xacro:dark_blue_material />
     </visual>
-    <collision>
-      <origin xyz="${position_screen}" rpy="0 0 ${pi/2}" />
-      <geometry>
-        <mesh filename="package://waver_description/meshes/oled_screen_link.stl" scale="${scale}" />
-      </geometry>
-    </collision>
   </link>
   <link name="wheel_back_left_link">
