Commit message: fix(description): world and robot physics improved

File: waver_description/urdf/depth_camera_zedxm.xacro (robot description, xacro)
@@ -6,5 +6,5 @@
         <inertial>
             <mass value="${zed_x_mini_mass}" />
-            <origin xyz="0 0 0" rpy="0 0 0" />
+            <origin xyz="-0.008213 0 0.015909" rpy="0 0 0" />
             <inertia ixx="1.2205537500280872e-05" iyy="4.073932956405751e-06" izz="1.3748504884318975e-05" ixy="0" iyz="0" ixz="0" />
         </inertial>
@@ -17,5 +17,5 @@
         </visual>
         <collision>
-            <origin xyz="0 0 ${base_to_top - 0.039}" rpy="0 0 0" />
+            <origin xyz="-0.008213 0 0.015909" rpy="0 0 0" />
             <geometry>
                 <box size="${zed_x_mini_dimensions}" />

File: waver_description/urdf/lidar.xacro (robot description, xacro)
@@ -6,5 +6,5 @@
         <inertial>
             <mass value="${mass_lidar}" />
-            <origin xyz="0 0 0" rpy="0 0 0" />
+            <origin xyz="-0.003726 0 -0.01135" rpy="0 0 ${pi/2}" />
             <inertia ixx="1.1969407982864896e-05" iyy="1.4912788506851203e-05" izz="1.9371239273809308e-05" ixy="0.0" iyz="0.0" ixz="0.0" />
         </inertial>
@@ -17,7 +17,7 @@
         </visual>
         <collision>
-            <origin xyz="0 0 -0.0107" rpy="0 0 0" />
+            <origin xyz="-0.003726 0 -0.01135" rpy="0 0 0" />
             <geometry>
-                <box size="0.0383 0.0383 0.030" />
+                <box size="0.04629 0.05395 0.0313" />
             </geometry>
         </collision>

File: waver_description/urdf/rasp_pi_camera.xacro (robot description, xacro)
@@ -4,4 +4,9 @@
     <xacro:include filename="$(find waver_description)/urdf/util.xacro" />
     <link name="rasp_pi_camera_link">
+        <inertial>
+            <mass value="${rasp_pi_camera_mass}" />
+            <origin xyz="0.005755 0 -0.011931" rpy="0 0 0" />
+            <inertia ixx="3.483652406539673e-07" iyy="2.047136044968006e-07" izz="2.209316971761668e-07" ixy="0" ixz="0" iyz="0" />
+        </inertial>
         <visual>
             <origin xyz="0 0.0125 0" rpy="0 0 ${-pi/2}" />
@@ -13,7 +18,7 @@
         </visual>
         <collision>
-            <origin xyz="0.005 0 -0.012" rpy="0 0 0" />
+            <origin xyz="0.005755 0 -0.011931" rpy="0 0 0" />
             <geometry>
-                <box size="0.01 0.025 0.023" />
+                <box size="0.01151 0.025 0.023862" />
             </geometry>
         </collision>

File: waver_description/urdf/util.xacro (robot description, xacro)
@@ -5,5 +5,5 @@
     <xacro:property name="scale" value="0.001 0.001 0.001" />
     <xacro:property name="floor_to_top" value="88.5e-03" />
-    <xacro:property name="floor_to_base" value="33.7e-03" />
+    <xacro:property name="floor_to_base" value="35.800994e-03" />
     <xacro:property name="base_to_top" value="${ floor_to_top - floor_to_base }" />
     <xacro:property name="length" value="183e-03" />
@@ -13,5 +13,5 @@
     <xacro:property name="pos_z_base" value="0.002703800678253174" />
     <xacro:property name="mass_base" value="0.110" />
-    <xacro:property name="mass_center_base" value="${pos_x_base} ${pos_y_base} ${pos_z_base}" />
+    <xacro:property name="mass_center_base" value="${-pos_y_base} ${pos_x_base} ${pos_z_base}" />
     <xacro:property name="position_base" value="${-pos_x_base} ${-pos_y_base} ${-pos_z_base}" />
     <!-- Top specifications -->
@@ -20,5 +20,5 @@
     <xacro:property name="pos_z_top" value="0.038709537506103515" />
     <xacro:property name="mass_top" value="0.326" />
-    <xacro:property name="mass_center_top" value="${pos_x_top} ${pos_y_top} ${pos_z_top}" />
+    <xacro:property name="mass_center_top" value="${-pos_y_top} ${pos_x_top} ${pos_z_top}" />
     <xacro:property name="position_top" value="${-pos_x_top} ${-pos_y_top} ${-pos_z_top}" />
     <!-- Accessories specifications -->
@@ -55,7 +55,10 @@
     <xacro:property name="positions_screen_joint" value="${-pos_y_screen} ${pos_x_screen} ${pos_z_screen}" />
     <!-- Wheels specifications -->
-    <xacro:property name="wheel_separation" value="123e-3" />
+    <xacro:property name="wheel_separation" value="130.673077e-3" />
     <xacro:property name="wheel_radius" value="40.6e-3" />
     <xacro:property name="wheel_width" value="42.5e-3" />
+    <xacro:property name="wheel_normal_force" value="1.8" />
+    <xacro:property name="wheel_slip_lateral" value="1.0" />
+    <xacro:property name="wheel_slip_longitudinal" value="0.0" />
     <!-- WBL specifications -->
     <xacro:property name="pos_x_wbl" value="0.06538582611083985" />
@@ -105,4 +108,4 @@
     <xacro:property name="zed_x_mini_mass" value="0.015" />
     <xacro:property name="zed_x_mini_scale" value="1 1 1" />
-    <xacro:property name="zed_x_mini_dimensions" value="0.030 0.093 0.0315" />
+    <xacro:property name="zed_x_mini_dimensions" value="0.0474 0.093552 0.031818" />
 </robot>

File: waver_description/urdf/waver.control.xacro (robot description, xacro)
@@ -41,4 +41,5 @@
         <mu1>0.8</mu1>
         <mu2>0.8</mu2>
+        <fdir1>0 0 1</fdir1>
         <selfCollide>false</selfCollide>
         <material>Gazebo/Black</material>
@@ -47,4 +48,5 @@
         <mu1>0.8</mu1>
         <mu2>0.8</mu2>
+        <fdir1>0 0 1</fdir1>
         <selfCollide>false</selfCollide>
         <material>Gazebo/Black</material>
@@ -53,4 +55,5 @@
         <mu1>0.8</mu1>
         <mu2>0.8</mu2>
+        <fdir1>0 0 1</fdir1>
         <selfCollide>false</selfCollide>
         <material>Gazebo/Black</material>
@@ -59,4 +62,5 @@
         <mu1>0.8</mu1>
         <mu2>0.8</mu2>
+        <fdir1>0 0 1</fdir1>
         <selfCollide>false</selfCollide>
         <material>Gazebo/Black</material>
@@ -71,4 +75,31 @@
         <plugin filename="libgz-sim-sensors-system.so" name="gz::sim::systems::Sensors">
             <render_engine>ogre2</render_engine>
+        </plugin>
+        <plugin filename="libgz-sim-wheel-slip-system.so"
+            name="gz::sim::systems::WheelSlip">
+            <wheel link_name="wheel_front_left_link">
+                <slip_compliance_lateral>${wheel_slip_lateral}</slip_compliance_lateral>
+                <slip_compliance_longitudinal>${wheel_slip_longitudinal}</slip_compliance_longitudinal>
+                <wheel_normal_force>${wheel_normal_force}</wheel_normal_force>
+                <wheel_radius>${wheel_radius}</wheel_radius>
+            </wheel>
+            <wheel link_name="wheel_front_right_link">
+                <slip_compliance_lateral>${wheel_slip_lateral}</slip_compliance_lateral>
+                <slip_compliance_longitudinal>${wheel_slip_longitudinal}</slip_compliance_longitudinal>
+                <wheel_normal_force>${wheel_normal_force}</wheel_normal_force>
+                <wheel_radius>${wheel_radius}</wheel_radius>
+            </wheel>
+            <wheel link_name="wheel_back_left_link">
+                <slip_compliance_lateral>${wheel_slip_lateral}</slip_compliance_lateral>
+                <slip_compliance_longitudinal>${wheel_slip_longitudinal}</slip_compliance_longitudinal>
+                <wheel_normal_force>${wheel_normal_force}</wheel_normal_force>
+                <wheel_radius>${wheel_radius}</wheel_radius>
+            </wheel>
+            <wheel link_name="wheel_back_right_link">
+                <slip_compliance_lateral>${wheel_slip_lateral}</slip_compliance_lateral>
+                <slip_compliance_longitudinal>${wheel_slip_longitudinal}</slip_compliance_longitudinal>
+                <wheel_normal_force>${wheel_normal_force}</wheel_normal_force>
+                <wheel_radius>${wheel_radius}</wheel_radius>
+            </wheel>
         </plugin>
     </gazebo>

File: waver_description/urdf/waver.gazebo.xacro (robot description, xacro)
@@ -41,4 +41,5 @@
     <mu1>0.8</mu1>
     <mu2>0.8</mu2>
+    <fdir1>0 0 1</fdir1>
     <selfCollide>false</selfCollide>
     <material>Gazebo/Black</material>
@@ -47,4 +48,5 @@
     <mu1>0.8</mu1>
     <mu2>0.8</mu2>
+    <fdir1>0 0 1</fdir1>
     <selfCollide>false</selfCollide>
     <material>Gazebo/Black</material>
@@ -53,4 +55,5 @@
     <mu1>0.8</mu1>
     <mu2>0.8</mu2>
+    <fdir1>0 0 1</fdir1>
     <selfCollide>false</selfCollide>
     <material>Gazebo/Black</material>
@@ -59,4 +62,5 @@
     <mu1>0.8</mu1>
     <mu2>0.8</mu2>
+    <fdir1>0 0 1</fdir1>
     <selfCollide>false</selfCollide>
     <material>Gazebo/Black</material>
@@ -70,4 +74,8 @@
       <wheel_separation>${wheel_separation}</wheel_separation>
       <wheel_radius>${wheel_radius}</wheel_radius>
+      <max_linear_velocity>0.3</max_linear_velocity>
+      <min_linear_velocity>-0.3</min_linear_velocity>
+      <max_angular_velocity>1.5</max_angular_velocity>
+      <min_angular_velocity>-1.5</min_angular_velocity>
       <max_linear_acceleration>2.0</max_linear_acceleration>
       <min_linear_acceleration>-2.0</min_linear_acceleration>
@@ -81,4 +89,31 @@
       <odom_publish_frequency>30</odom_publish_frequency>
     </plugin>
+    <plugin filename="libgz-sim-wheel-slip-system.so"
+      name="gz::sim::systems::WheelSlip">
+      <wheel link_name="wheel_front_left_link">
+        <slip_compliance_lateral>${wheel_slip_lateral}</slip_compliance_lateral>
+        <slip_compliance_longitudinal>${wheel_slip_longitudinal}</slip_compliance_longitudinal>
+        <wheel_normal_force>${wheel_normal_force}</wheel_normal_force>
+        <wheel_radius>${wheel_radius}</wheel_radius>
+      </wheel>
+      <wheel link_name="wheel_front_right_link">
+        <slip_compliance_lateral>${wheel_slip_lateral}</slip_compliance_lateral>
+        <slip_compliance_longitudinal>${wheel_slip_longitudinal}</slip_compliance_longitudinal>
+        <wheel_normal_force>${wheel_normal_force}</wheel_normal_force>
+        <wheel_radius>${wheel_radius}</wheel_radius>
+      </wheel>
+      <wheel link_name="wheel_back_left_link">
+        <slip_compliance_lateral>${wheel_slip_lateral}</slip_compliance_lateral>
+        <slip_compliance_longitudinal>${wheel_slip_longitudinal}</slip_compliance_longitudinal>
+        <wheel_normal_force>${wheel_normal_force}</wheel_normal_force>
+        <wheel_radius>${wheel_radius}</wheel_radius>
+      </wheel>
+      <wheel link_name="wheel_back_right_link">
+        <slip_compliance_lateral>${wheel_slip_lateral}</slip_compliance_lateral>
+        <slip_compliance_longitudinal>${wheel_slip_longitudinal}</slip_compliance_longitudinal>
+        <wheel_normal_force>${wheel_normal_force}</wheel_normal_force>
+        <wheel_radius>${wheel_radius}</wheel_radius>
+      </wheel>
+    </plugin>
     <plugin filename="libgz-sim-joint-state-publisher-system.so"
       name="gz::sim::systems::JointStatePublisher">

File: waver_description/urdf/waver.xacro (robot description, xacro)
@@ -27,5 +27,5 @@
       <mass value="${mass_base}" />
       <origin xyz="${mass_center_base}" rpy="0 0 ${pi/2}" />
-      <inertia ixx="0.00024519341275127564" iyy="0.0001572047252476648" izz="0.0001572047252476648"
+      <inertia ixx="0.00024519341275127564" iyy="0.0001572047252476648" izz="0.0003954468754399687"
         ixy="0.0" iyz="0.0" ixz="0.0" />
     </inertial>
@@ -38,7 +38,7 @@
     </visual>
     <collision>
-      <origin xyz="0 0 0" rpy="0 0 ${pi/2}" />
-      <geometry>
-        <mesh filename="package://waver_description/meshes/base_link.stl" scale="${scale}" />
+      <origin xyz="0.000001 0.000049626 0.006036" rpy="0 0 0" />
+      <geometry>
+        <box size="0.162386 0.129501 0.019472" />
       </geometry>
     </collision>
@@ -59,7 +59,7 @@
     </visual>
     <collision>
-      <origin xyz="0 0 0" rpy="0 0 ${pi/2}" />
-      <geometry>
-        <mesh filename="package://waver_description/meshes/top_shell_link.stl" scale="${scale}" />
+      <origin xyz="0.000001 -0.000001 0.025578" rpy="0 0 0" />
+      <geometry>
+        <box size="0.183106 0.163738 0.054312" />
       </geometry>
     </collision>
@@ -74,7 +74,7 @@
     </visual>
     <collision>
-      <origin xyz="${position_acces}" rpy="0 0 ${pi/2}" />
-      <geometry>
-        <mesh filename="package://waver_description/meshes/accessories_link.stl" scale="${scale}" />
+      <origin xyz="-0.001662418 0.022091042 0.001653101" rpy="0 0 0" />
+      <geometry>
+        <box size="0.027758 0.065151 0.027758" />
       </geometry>
     </collision>
@@ -189,5 +189,5 @@
   <joint
     name="base_joint" type="fixed">
-    <origin xyz="0.0 0.0 33.7e-3" rpy="0 0 0" />
+    <origin xyz="0 0 ${floor_to_base}" rpy="0 0 0" />
     <parent link="base_footprint" />
     <child link="base_link" />
@@ -218,4 +218,5 @@
     <child link="wheel_back_left_link" />
     <axis xyz="0 1 0" />
+    <limit effort="0.07" velocity="10.0" />
   </joint>
   <joint name="wheel_front_left_joint" type="continuous">
@@ -224,4 +225,5 @@
     <child link="wheel_front_left_link" />
     <axis xyz="0 1 0" />
+    <limit effort="0.07" velocity="10.0" />
   </joint>
   <joint name="wheel_front_right_joint" type="continuous">
@@ -230,4 +232,5 @@
     <child link="wheel_front_right_link" />
     <axis xyz="0 1 0" />
+    <limit effort="0.07" velocity="10.0" />
   </joint>
   <joint name="wheel_back_right_joint" type="continuous">
@@ -236,4 +239,5 @@
     <child link="wheel_back_right_link" />
     <axis xyz="0 1 0" />
+    <limit effort="0.07" velocity="10.0" />
   </joint>
 </robot>
