Commit message: fix(description): angular and linear velocity values improved

File: waver_description/urdf/waver.control.xacro (robot description, xacro)
@@ -110,6 +110,6 @@
         <joint name="wheel_front_left_joint">
             <command_interface name="velocity">
-                <param name="min">-10</param>
-                <param name="max">10</param>
+                <param name="min">-40.0</param>
+                <param name="max">40.0</param>
             </command_interface>
             <state_interface name="position" />
@@ -118,6 +118,6 @@
         <joint name="wheel_front_right_joint">
             <command_interface name="velocity">
-                <param name="min">-10</param>
-                <param name="max">10</param>
+                <param name="min">-40.0</param>
+                <param name="max">40.0</param>
             </command_interface>
             <state_interface name="position" />
@@ -126,6 +126,6 @@
         <joint name="wheel_back_left_joint">
             <command_interface name="velocity">
-                <param name="min">-10.0</param>
-                <param name="max">10.0</param>
+                <param name="min">-40.0</param>
+                <param name="max">40.0</param>
             </command_interface>
             <state_interface name="position" />
@@ -134,6 +134,6 @@
         <joint name="wheel_back_right_joint">
             <command_interface name="velocity">
-                <param name="min">-10.0</param>
-                <param name="max">10.0</param>
+                <param name="min">-40.0</param>
+                <param name="max">40.0</param>
             </command_interface>
             <state_interface name="position" />

File: waver_description/urdf/waver.gazebo.xacro (robot description, xacro)
@@ -74,12 +74,12 @@
       <wheel_separation>${wheel_separation}</wheel_separation>
       <wheel_radius>${wheel_radius}</wheel_radius>
-      <max_linear_velocity>0.3</max_linear_velocity>
-      <min_linear_velocity>-0.3</min_linear_velocity>
-      <max_angular_velocity>1.5</max_angular_velocity>
-      <min_angular_velocity>-1.5</min_angular_velocity>
+      <max_linear_velocity>1.25</max_linear_velocity>
+      <min_linear_velocity>-1.25</min_linear_velocity>
+      <max_angular_velocity>${1.5 * pi}</max_angular_velocity>
+      <min_angular_velocity>${-1.5 * pi}</min_angular_velocity>
       <max_linear_acceleration>2.0</max_linear_acceleration>
       <min_linear_acceleration>-2.0</min_linear_acceleration>
-      <max_angular_acceleration>4.0</max_angular_acceleration>
-      <min_angular_acceleration>-4.0</min_angular_acceleration>
+      <max_angular_acceleration>7.5</max_angular_acceleration>
+      <min_angular_acceleration>-7.5</min_angular_acceleration>
       <topic>cmd_vel</topic>
       <odom_topic>odometry</odom_topic>

File: waver_description/urdf/waver.xacro (robot description, xacro)
@@ -218,5 +218,5 @@
     <child link="wheel_back_left_link" />
     <axis xyz="0 1 0" />
-    <limit effort="0.07" velocity="10.0" />
+    <limit effort="0.15" velocity="40.0" />
   </joint>
   <joint name="wheel_front_left_joint" type="continuous">
@@ -225,5 +225,5 @@
     <child link="wheel_front_left_link" />
     <axis xyz="0 1 0" />
-    <limit effort="0.07" velocity="10.0" />
+    <limit effort="0.15" velocity="40.0" />
   </joint>
   <joint name="wheel_front_right_joint" type="continuous">
@@ -232,5 +232,5 @@
     <child link="wheel_front_right_link" />
     <axis xyz="0 1 0" />
-    <limit effort="0.07" velocity="10.0" />
+    <limit effort="0.15" velocity="40.0" />
   </joint>
   <joint name="wheel_back_right_joint" type="continuous">
@@ -239,5 +239,5 @@
     <child link="wheel_back_right_link" />
     <axis xyz="0 1 0" />
-    <limit effort="0.07" velocity="10.0" />
+    <limit effort="0.15" velocity="40.0" />
   </joint>
 </robot>
